File: nes_power_video.kicad_sch (KiCad schematic)
At the start: 23 parts, among them J2 Audio, J3 Video, J4 Conn_01x05, J5 RGB conn feed, Q1 2SA733, U1 TPS2553DBV

Commit message: feat(bom): carry sourcing metadata on the board, and split out an SMD-only fab package
The PCBWay BOM is exported from the board, but every sourcing field lived only
on the schematic symbols, so the MPN column came out empty for all but J2 and
J3 — and those two only because they still carried the legacy
Manufacturer_Part_Number field. MPN is the field PCBWay sources by, so the
package could not have been assembled as exported.

Copy Manufacturer, MPN, LCSC, Spec, Supplier Link, Datasheet and Description
from the schematic into the matching footprints. KiCad does this from the GUI's
"Update PCB from Schematic"; kicad-cli has no equivalent, so the fields are
written into the board s-expression directly, hidden on F.Fab. Board geometry
is byte-identical after stripping properties — no copper moved.

This also flushes out v1 identities the board was still holding: D1's datasheet
pointed at Vishay's 15KE part rather than the fitted Littelfuse 1.5KE6.8A, and
Q1's at the 2SA1015 it no longer is. Schematic parity findings go 27 to 0.

TP1-TP4 become in_bom no on the schematic, matching what the board already
said. They are bare plated holes, not purchased parts.

Add tools/pcbway_assembly.py, which turns a gate package into the SMD-only
upload pair. It reads mount type from the board's own (attr ...) and pad list
rather than a list of designators, so a part that changes mounting cannot keep
its old side of the split, and it refuses to write when an SMD part has no MPN.

Two findings it surfaces, both recorded in docs/pcbway-smd-assembly.md:

USB-C1 is Hybrid rather than SMD. Four of its ten pads are through-hole shell
stakes sitting on F.Paste — pin-in-paste, reflowing with the SMD pass. Labelled
SMD, an assembler would reasonably place the part and leave the four mechanical
anchors dry, leaving the connector that takes the insertion force held on by six
0.7 mm signal pads.

U1 (TPS2553DBVR) has no Western stock: DigiKey 0 across all pack types, Mouser 0
with a 112-day fac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
Parts:
- TP1, TP2, TP3, TP4: now left out of the parts list
Changed lines of the file:
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@@
 		(body_style 1)
 		(exclude_from_sim no)
-		(in_bom yes)
+		(in_bom no)
 		(on_board yes)
 		(in_pos_files yes)
@@
 		(body_style 1)
 		(exclude_from_sim no)
-		(in_bom yes)
+		(in_bom no)
 		(on_board yes)
 		(in_pos_files yes)
@@
 		(body_style 1)
 		(exclude_from_sim no)
-		(in_bom yes)
+		(in_bom no)
 		(on_board yes)
 		(in_pos_files yes)
@@
 		(body_style 1)
 		(exclude_from_sim no)
-		(in_bom yes)
-		(on_board yes)
-		(in_pos_files yes)
+		(in_bom no)
+		(on_board yes)
+		(in_pos_files yes)

Commit message: sourcing(v2): move USB-C1, F1 and D1 to LCSC parts
Closes the last non-LCSC lines on the v2 BOM so the whole SMD assembly
BOM can be sourced from one place, which is what U1's Western stockout
forced in the first place.

USB-C1: GCT USB4970-00-A -> USB4125-GF-A-0190 (LCSC C5246813).
LCSC does not stock the USB4970 at all, so searching that MPN was always
going to come up empty. The USB4125 is a different GCT line number that
LCSC does carry, and the board was already laid out to its land pattern
-- the KiCad footprints for USB4125-xx-x and USB4125-xx-x-0190 are
byte-identical in copper, silk, fab, courtyard and drills, differing only
in name, descr and 3D model. Verified against GCT's own drawing: pad
centres 1.00/3.04/5.50 mm, shell holes 8.64 x 3.80 mm, and the ordering
table's "Blank = 1.00mm, 0190 = 1.90mm" stake codes. The -0190 is chosen
because its 1.90 mm stake protrudes 0.30 mm through this 1.6 mm board and
gives a bottom-side fillet, where the 1.00 mm stake does not reach through.
No layout change: zero copper or geometry lines differ.

F1: Littelfuse RHEF200 -> Jinrui JK30-200 (LCSC C369104).
LCSC does not stock the RHEF series. IH 2.0 A unchanged, IT 3.8 -> 4.0 A,
resistance improves slightly (40/100 mOhm vs 45/110), 30 V rather than
16 V, Imax 100 -> 40 A. Confirmed radial leaded from the JK30 datasheet:
D(typ) lead spacing 5.1 mm, tinned 24AWG/0.5 mm leads, C(max) 3.0 mm body
thickness, all consistent with the Bourns MF-RG300 land pattern F1 borrows.

The JKSEMI JK16-200T (C5183874) was evaluated first and rejected: LCSC
lists it as Through Hole P=5.1mm, but its own datasheet is headed "JK16
Series Surface Mount PTC Devices" and LCSC has no land pattern drawn for
it. The package could not be confirmed, so it is called out as a
do-not-substitute in both BOM.csv and the README.

D1: LCSC C294199 added as a second source. That stock is DOWO-branded
(VWM 5.8 V, VBR 6.46 V, VC 10.5 V @ 142.86 A), equivalent to the
Littelfuse figures the design was character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
Parts:
- D1: BOM Comments (none) -> LCSC stock of the 1.5KE6.8A is DOWO-branded (C294199, DO-20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; LCSC (none) -> C294199
- F1: BOM Comments (none) -> Replaces Littelfuse RHEF200, which LCSC does not stock. IH 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; Footprint Note No Littelfuse RHEF footprint exists in the KiCad libraries.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 -> No JK30 footprint exists in the KiCad libraries. F1 uses th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; LCSC (none) -> C369104; MPN RHEF200 -> JK30-200; Manufacturer Littelfuse -> Jinrui (ShenZhen JinRui Electronic Material); Spec PPTC radial, IH 2.0 A / IT 3.8 A / 16 V max -> PPTC radial leaded, IH 2.0 A / IT 4.0 A / 30 V max / Imax 4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; Supplier Link https://www.digikey.com/en/products/detail/littelfuse-inc/R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 -> https://www.lcsc.com/product-detail/C369104.html
- USB-C1: value USB4970-00-A -> USB4125-GF-A-0190; footprint Connector_USB:USB_C_Receptacle_GCT_USB4125-xx-x_6P_TopMnt_Horizontal -> Connector_USB:USB_C_Receptacle_GCT_USB4125-xx-x-0190_6P_TopMnt_Horizontal; BOM Comments (none) -> Replaces GCT USB4970-00-A, which LCSC does not stock - an M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; Footprint Note KiCad has no USB4970 footprint. GCT's USB4970 drawing speci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 -> Exact KiCad footprint for this MPN. USB_C_Receptacle_GCT_US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; LCSC (none) -> C5246813; MPN USB4970-00-A -> USB4125-GF-A-0190; Manufacturer GCT -> Global Connector Technology (GCT); Spec USB Type-C receptacle, 6P power-only (VBUS x2, GND x2, CC1, CC2) -> USB Type-C receptacle, 6P power-only (VBUS x2, GND x2, CC1, CC2), 48 V / 3 A, 20,000 mating cycles, 1.90 mm shell stake; Supplier Link https://www.digikey.com/en/products/detail/gct/USB4970-00-A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 -> https://www.lcsc.com/product-detail/C5246813.html
Changed lines of the file:
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@@
 			)
 		)
-		(property "Datasheet" "https://www.littelfuse.com/assetdocs/resettable-ptc-rhef-datasheet?assetguid=5c5a29fe-1611-4d65-b4ce-dc979c44d206"
+		(property "Datasheet" "https://www.lcsc.com/datasheet/C369104.pdf"
 			(at 128.27 143.51 0)
 			(hide yes)
@@
 			)
 		)
-		(property "Manufacturer" "Littelfuse"
+		(property "Manufacturer" "Jinrui (ShenZhen JinRui Electronic Material)"
 			(at 128.27 143.51 0)
 			(hide yes)
@@
 			)
 		)
-		(property "MPN" "RHEF200"
+		(property "MPN" "JK30-200"
 			(at 128.27 143.51 0)
 			(hide yes)
@@
 			)
 		)
-		(property "Spec" "PPTC radial, IH 2.0 A / IT 3.8 A / 16 V max"
+		(property "Spec" "PPTC radial leaded, IH 2.0 A / IT 4.0 A / 30 V max / Imax 40 A, Rmin 40 mOhm, R1max 100 mOhm, trip 11 s max, 5.1 mm lead pitch, 0.5 mm (24AWG) leads, 3.0 mm body thickness, 15.2 mm max height"
 			(at 128.27 143.51 0)
 			(hide yes)
@@
 			)
 		)
-		(property "Supplier Link" "https://www.digikey.com/en/products/detail/littelfuse-inc/RHEF200/5130265"
+		(property "Supplier Link" "https://www.lcsc.com/product-detail/C369104.html"
 			(at 128.27 143.51 0)
 			(hide yes)
@@
 			)
 		)
-		(property "Footprint Note" "No Littelfuse RHEF footprint exists in the KiCad libraries. F1 uses the Bourns MF-RG300 land pattern: pads at (0,0) and (5.1,1.2), 5.24 mm centre-to-centre, 1.01 mm drills. RHEF200 leads are 0.51 mm dia at 5.05 +/-0.75 mm spacing, so they fit, but the Bourns part is a 3.0 A/5.1 A device and the drawn body outline is its, not the RHEF200's - do not trust the outline for clearance."
+		(property "Footprint Note" "No JK30 footprint exists in the KiCad libraries. F1 uses the Bourns MF-RG300 land pattern: pads at (0,0) and (5.1,1.2), 5.24 mm centre-to-centre, 1.01 mm drills. Confirmed against the JK30 datasheet: the series is radial leaded, D(typ) lead spacing is 5.1 mm and leads are tinned 24AWG / 0.5 mm dia across the whole family, so they seat in the 1.01 mm drills with the same slight splay onto the diagonal pad pair that the RHEF200 needed. C(max) body thickness is 3.0 mm, matching the footprint's 3.0 mm in-plane depth. The silkscreen outline is still the Bourns 3.0 A/5.1 A body, not this part's - do not use it for clearance."
 			(at 128.27 143.51 0)
 			(hide yes)
@@
 					(size 1.27 1.27)
 				)
+			)
+		)
+		(property "BOM Comments" "Replaces Littelfuse RHEF200, which LCSC does not stock. IH 2.0 A unchanged; IT rises 3.8 A -> 4.0 A; resistance improves slightly (Rmin 40 / R1max 100 mOhm vs the RHEF200's 45/110), so marginally less drop on the 5 V rail. Imax drops 100 A -> 40 A: that is the maximum fault current the device can interrupt, and a USB-C source limited to ~3 A never approaches it. CHECK HEIGHT BEFORE ORDERING: B(max) is 15.2 mm against the RHEF200's ~9-10 mm, and radial PPTCs stand vertically, so this is ~5-6 mm more height above the board inside the NES shell. F1 sits 7.2 mm from the top board edge. Sourcing checked 2026-09-09: 5,800 in stock, MOQ 10, multiple 10, $0.063 at qty 10. NOT the JKSEMI JK16-200T (C5183874): LCSC lists that part as Through Hole P=5.1mm, but its own datasheet is headed 'JK16 Series Surface Mount PTC Devices' and LCSC has no land pattern drawn for it, so its package could not be confirmed - do not substitute it without checking the mechanical drawing." (at 0 0 0)
+			(effects
+				(font
+					(size 1.27 1.27)
+				)
+				(hide yes)
+			)
+		)
+		(property "LCSC" "C369104" (at 0 0 0)
+			(effects
+				(font
+					(size 1.27 1.27)
+				)
+				(hide yes)
 			)
 		)
@@
 			)
 		)
+		(property "BOM Comments" "LCSC stock of the 1.5KE6.8A is DOWO-branded (C294199, DO-201, MOQ 5): VWM 5.8 V, VBR 6.46 V, VC 10.5 V @ 142.86 A - equivalent to the Littelfuse figures this design was characterised against, so every conclusion in the README still holds, including the finding that D1 does not protect U1. Manufacturer/MPN fields still name Littelfuse because that is the part actually fitted on v1 and the one the DigiKey supplier link points at; 1.5KE6.8A is a generic type number, not a Littelfuse-only MPN. Order either." (at 0 0 0)
+			(effects
+				(font
+					(size 1.27 1.27)
+				)
+				(hide yes)
+			)
+		)
+		(property "LCSC" "C294199" (at 0 0 0)
+			(effects
+				(font
+					(size 1.27 1.27)
+				)
+				(hide yes)
+			)
+		)
 		(pin "1"
 		)
@@
 			)
 		)
-		(property "Value" "USB4970-00-A"
+		(property "Value" "USB4125-GF-A-0190"
 			(at 113.538 132.842 0)
 			(show_name no)
@@
 			)
 		)
-		(property "Footprint" "Connector_USB:USB_C_Receptacle_GCT_USB4125-xx-x_6P_TopMnt_Horizontal"
+		(property "Footprint" "Connector_USB:USB_C_Receptacle_GCT_USB4125-xx-x-0190_6P_TopMnt_Horizontal"
 			(at 116.84 151.13 0)
 			(hide yes)
@@
 			)
 		)
-		(property "Datasheet" "https://gct.co/files/drawings/usb4970.pdf"
+		(property "Datasheet" "https://gct.co/files/drawings/usb4125.pdf"
 			(at 113.03 153.67 0)
 			(hide yes)
@@
 			)
 		)
-		(property "Manufacturer" "GCT"
+		(property "Manufacturer" "Global Connector Technology (GCT)"
 			(at 113.03 153.67 0)
 			(hide yes)
@@
 			)
 		)
-		(property "MPN" "USB4970-00-A"
+		(property "MPN" "USB4125-GF-A-0190"
 			(at 113.03 153.67 0)
 			(hide yes)
@@
 			)
 		)
-		(property "Spec" "USB Type-C receptacle, 6P power-only (VBUS x2, GND x2, CC1, CC2)"
+		(property "Spec" "USB Type-C receptacle, 6P power-only (VBUS x2, GND x2, CC1, CC2), 48 V / 3 A, 20,000 mating cycles, 1.90 mm shell stake"
 			(at 113.03 153.67 0)
 			(hide yes)
@@
 			)
 		)
-		(property "Supplier Link" "https://www.digikey.com/en/products/detail/gct/USB4970-00-A/28722813"
+		(property "Supplier Link" "https://www.lcsc.com/product-detail/C5246813.html"
 			(at 113.03 153.67 0)
 			(hide yes)
@@
 			)
 		)
-		(property "Footprint Note" "KiCad has no USB4970 footprint. GCT's USB4970 drawing specifies the same recommended layout as the USB4125: pad centres 1.00/3.04/5.50 mm, widths 0.70/0.76/0.80 mm x 1.20 mm, shell holes 8.64 x 3.80 mm apart, 1.10 x 1.70 mm with 0.60 x 1.20 mm slots. Verified against the drawing 2026-08-28. USB4970-00-A takes the 1.00 mm shell stake, so the plain USB4125-xx-x footprint is the match; -0190 is the 1.90 mm stake variant."
+		(property "Footprint Note" "Exact KiCad footprint for this MPN. USB_C_Receptacle_GCT_USB4125-xx-x-0190 is byte-identical in copper, silk, fab, courtyard and drills to the plain USB4125-xx-x land pattern the board was laid out with - only the name, descr and 3D model differ - so this is a naming correction, not a layout change. The -0190 suffix is the 1.90 mm shell stake, which protrudes 0.30 mm through a 1.6 mm board and gives a bottom-side fillet; the 1.00 mm stake (plain USB4125-GF-A, LCSC C3151650) does not reach through."
 			(at 113.03 153.67 0)
 			(hide yes)
@@
 			)
 		)
+		(property "BOM Comments" "Replaces GCT USB4970-00-A, which LCSC does not stock - an MPN search will always come up empty. The USB4125 is a different GCT line number that LCSC does carry, and the board was already laid out to its land pattern. Stock is thin (~600-3,700 depending on source) next to the generic Chinese 6P parts, so order spares. Plain 1.00 mm stake variant is C3151650 if the -0190 is out." (at 0 0 0)
+			(effects
+				(font
+					(size 1.27 1.27)
+				)
+				(hide yes)
+			)
+		)
+		(property "LCSC" "C5246813" (at 0 0 0)
+			(effects
+				(font
+					(size 1.27 1.27)
+				)
+				(hide yes)
+			)
+		)

Commit message: sourcing(v2): keep the RHEF200 for F1 rather than moving it to LCSC
F1 does not belong in the LCSC consolidation. The constraint that drove
this was U1 being unobtainable in the West, which matters because PCBWay
sources the SMD assembly BOM -- C3, R6, U1, USB-C1 -- from one supplier.
F1 is through-hole and is not on that BOM. Neither is D1. Both are hand
-fitted parts that can come from anywhere, and a Mouser order is happening
regardless because the Switchcraft RCA jacks are not an LCSC line and
never will be.

The RHEF200 is also simply the better part. Against the closest LCSC
alternative, Jinrui JK30-200: Imax 100 A vs 40 A, trip 3.8 A vs 4.0 A,
body ~9-10 mm vs 15.2 mm. The only gain was R1max 110 -> 100 mOhm, which
is noise on a rail that drops ~130 mV at U1's limit either way.

F1 on this build is desoldered from the v1 board and reused, so nothing is
being ordered for it at all.

Reverts the advisory and the simulation harness to their pre-change state:
both are byte-identical to c020073, since the only reason they moved was
F1's trip current. The advisory goes back to a single-part story at 3.8 A,
which is accurate for every board that exists.

BOM.csv and the README now record why F1 is deliberately not an LCSC line,
and carry the JK16-200T package warning for whoever looks next.

USB-C1 and D1 from 05584b2 are unaffected.

Verified: ERC 0 violations; DRC 0 unconnected, 0 schematic parity issues,
6 pre-existing silkscreen warnings; no copper or geometry change vs c020073.

Co-Authored-By: Claude Opus 5 <noreply@anthropic.com>
Claude-Session: https://claude.ai/code/session_011og7T5AvxjjAMvr7XwQ3K1
Parts:
- F1: BOM Comments Replaces Littelfuse RHEF200, which LCSC does not stock. IH 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 -> Reused from the v1 build - desoldered, not reordered. Delib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; Footprint Note No JK30 footprint exists in the KiCad libraries. F1 uses th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 -> No Littelfuse RHEF footprint exists in the KiCad libraries.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; LCSC C369104 -> (none); MPN JK30-200 -> RHEF200; Manufacturer Jinrui (ShenZhen JinRui Electronic Material) -> Littelfuse; Spec PPTC radial leaded, IH 2.0 A / IT 4.0 A / 30 V max / Imax 4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 -> PPTC radial, IH 2.0 A / IT 3.8 A / 16 V max / Imax 100 A, R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; Supplier Link https://www.lcsc.com/product-detail/C369104.html -> https://www.digikey.com/en/products/detail/littelfuse-inc/R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
Changed lines of the file:
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@@
 			)
 		)
-		(property "Datasheet" "https://www.lcsc.com/datasheet/C369104.pdf"
+		(property "Datasheet" "https://www.littelfuse.com/assetdocs/resettable-ptc-rhef-datasheet?assetguid=5c5a29fe-1611-4d65-b4ce-dc979c44d206"
 			(at 128.27 143.51 0)
 			(hide yes)
@@
 			)
 		)
-		(property "Manufacturer" "Jinrui (ShenZhen JinRui Electronic Material)"
+		(property "Manufacturer" "Littelfuse"
 			(at 128.27 143.51 0)
 			(hide yes)
@@
 			)
 		)
-		(property "MPN" "JK30-200"
+		(property "MPN" "RHEF200"
 			(at 128.27 143.51 0)
 			(hide yes)
@@
 			)
 		)
-		(property "Spec" "PPTC radial leaded, IH 2.0 A / IT 4.0 A / 30 V max / Imax 40 A, Rmin 40 mOhm, R1max 100 mOhm, trip 11 s max, 5.1 mm lead pitch, 0.5 mm (24AWG) leads, 3.0 mm body thickness, 15.2 mm max height"
+		(property "Spec" "PPTC radial, IH 2.0 A / IT 3.8 A / 16 V max / Imax 100 A, Rmin 45 mOhm, R1max 110 mOhm"
 			(at 128.27 143.51 0)
 			(hide yes)
@@
 			)
 		)
-		(property "Supplier Link" "https://www.lcsc.com/product-detail/C369104.html"
+		(property "Supplier Link" "https://www.digikey.com/en/products/detail/littelfuse-inc/RHEF200/5130265"
 			(at 128.27 143.51 0)
 			(hide yes)
@@
 			)
 		)
-		(property "Footprint Note" "No JK30 footprint exists in the KiCad libraries. F1 uses the Bourns MF-RG300 land pattern: pads at (0,0) and (5.1,1.2), 5.24 mm centre-to-centre, 1.01 mm drills. Confirmed against the JK30 datasheet: the series is radial leaded, D(typ) lead spacing is 5.1 mm and leads are tinned 24AWG / 0.5 mm dia across the whole family, so they seat in the 1.01 mm drills with the same slight splay onto the diagonal pad pair that the RHEF200 needed. C(max) body thickness is 3.0 mm, matching the footprint's 3.0 mm in-plane depth. The silkscreen outline is still the Bourns 3.0 A/5.1 A body, not this part's - do not use it for clearance."
+		(property "Footprint Note" "No Littelfuse RHEF footprint exists in the KiCad libraries. F1 uses the Bourns MF-RG300 land pattern: pads at (0,0) and (5.1,1.2), 5.24 mm centre-to-centre, 1.01 mm drills. RHEF200 leads are 0.51 mm dia at 5.05 +/-0.75 mm spacing, so they fit, but the Bourns part is a 3.0 A/5.1 A device and the drawn body outline is its, not the RHEF200's - do not trust the outline for clearance."
 			(at 128.27 143.51 0)
 			(hide yes)
@@
 			)
 		)
-		(property "BOM Comments" "Replaces Littelfuse RHEF200, which LCSC does not stock. IH 2.0 A unchanged; IT rises 3.8 A -> 4.0 A; resistance improves slightly (Rmin 40 / R1max 100 mOhm vs the RHEF200's 45/110), so marginally less drop on the 5 V rail. Imax drops 100 A -> 40 A: that is the maximum fault current the device can interrupt, and a USB-C source limited to ~3 A never approaches it. CHECK HEIGHT BEFORE ORDERING: B(max) is 15.2 mm against the RHEF200's ~9-10 mm, and radial PPTCs stand vertically, so this is ~5-6 mm more height above the board inside the NES shell. F1 sits 7.2 mm from the top board edge. Sourcing checked 2026-09-09: 5,800 in stock, MOQ 10, multiple 10, $0.063 at qty 10. NOT the JKSEMI JK16-200T (C5183874): LCSC lists that part as Through Hole P=5.1mm, but its own datasheet is headed 'JK16 Series Surface Mount PTC Devices' and LCSC has no land pattern drawn for it, so its package could not be confirmed - do not substitute it without checking the mechanical drawing." (at 0 0 0)
+		(property "BOM Comments" "Reused from the v1 build - desoldered, not reordered. Deliberately NOT moved to LCSC: F1 is through-hole, so it is not on the SMD assembly BOM PCBWay sources, and the Littelfuse part is better than the LCSC alternatives on every axis that matters (Imax 100 A vs 40 A, 3.8 A trip vs 4.0 A, ~9-10 mm body vs 15.2 mm). If it ever does need reordering, buy it from DigiKey or Mouser alongside the Switchcraft RCA jacks, which cannot come from LCSC either. The closest LCSC parts are Jinrui JK30-200 (C369104, verified radial, but taller and only 40 A Imax) and JKSEMI JK16-200T (C5183874, whose datasheet is headed 'Surface Mount' despite LCSC listing it as through-hole - package unconfirmed, do not use without checking the mechanical drawing)." (at 0 0 0)
 			(effects
 				(font
@@
 			)
 		)
-		(property "LCSC" "C369104" (at 0 0 0)
+		(property "LCSC" "" (at 0 0 0)
 			(effects
 				(font
